File: ym3812_card_with_gameport/ym3812_card_with_gameport.kicad_pcb (KiCad board)
At the start: 2 copper layers, 115.6 x 106.7 mm, 81 parts, among them IC1 74LS138, IC11 NE558, IC12 74HCT02, IC13 74LS74, IC18 74LS244, IC2 74LS138, IC3 74LS138, IC4 74LS245, IC6 YM3812, IC7 Y3014B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

Commit message: mark R5, R6, R7 and R8 as DNP
Parts:
- R5, R6, R7, R8: value ? -> DNP
Changed lines of the file:
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@@
       (effects (font (size 1 1) (thickness 0.15)) (justify mirror))
     )
-    (fp_text value ? (at 0 -1.82 90) (layer B.Fab)
+    (fp_text value DNP (at 0 -1.82 90) (layer B.Fab)
       (effects (font (size 1 1) (thickness 0.15)) (justify mirror))
     )
@@
       (effects (font (size 1 1) (thickness 0.15)) (justify mirror))
     )
-    (fp_text value ? (at 0 -1.82 90) (layer B.Fab)
+    (fp_text value DNP (at 0 -1.82 90) (layer B.Fab)
       (effects (font (size 1 1) (thickness 0.15)) (justify mirror))
     )
@@
       (effects (font (size 1 1) (thickness 0.15)) (justify mirror))
     )
-    (fp_text value ? (at 0 -1.82 90) (layer B.Fab)
+    (fp_text value DNP (at 0 -1.82 90) (layer B.Fab)
       (effects (font (size 1 1) (thickness 0.15)) (justify mirror))
     )
@@
       (effects (font (size 1 1) (thickness 0.15)) (justify mirror))
     )
-    (fp_text value ? (at 0 -1.82 90) (layer B.Fab)
+    (fp_text value DNP (at 0 -1.82 90) (layer B.Fab)
       (effects (font (size 1 1) (thickness 0.15)) (justify mirror))
     )
